Commit message: added xacro

File: robo.urdf (robot description, URDF)
Before this commit: robot robo, 5 links, 4 joints
Links:
- link base_link: geometry visual box size=${base_length} ${base_width} ${base_height}
- link left_wheel: geometry visual cylinder length=${wheel_length} radius=${wheel_radius}
- link right_wheel: geometry visual cylinder length=${wheel_length} radius=${wheel_radius}
Joints:
- joint caster_base: origin xyz=0.2 0 -0.05 rpy=0 0 0 -> xyz=${base_length/3.0} 0 ${-wheel_radius/2.0} rpy=0 0 0
- joint footprint: origin xyz=0 0 0.1 rpy=0 0 0 -> xyz=0 0 ${wheel_radius} rpy=0 0 0
- joint left_wheel_base: origin xyz=-0.15 0.225 0 rpy=0 0 0 -> xyz=${-base_length/4.0} ${(base_width+wheel_length)/2.0} 0 rpy=0 0 0
- joint right_wheel_base: origin xyz=-0.15 -0.225 0 rpy=0 0 0 -> xyz=${-base_length/4.0} ${-(base_width+wheel_length)/2.0} 0 rpy=0 0 0

Commit message: xacro and macros added

File: robo.urdf (robot description, URDF)
Before this commit: robot robo, 5 links, 4 joints
Links:
- removed link left_wheel
- removed link right_wheel
